Commit message: added k3lso urdf to rex urdf
added k3lso urdf to rex urdf. changed a few things. still not working as it shohuld

File: rex_gym/util/pybullet_data/assets/urdf/rex.urdf (robot description, URDF)
Before this commit: robot rex, 23 links, 22 joints
Links:
- removed link chassis_front_link
- removed link chassis_rear_link
- link base_link: mass 1.20 -> 10.0; geometry collision mesh filename=stl/base_link.stl scale=0.001 0.001 0.001; visual mesh filename=stl/base_link.stl scale=0.001 0.001 0.001
- link front_left_foot_link: mass 0.1 -> 0.11741117146712181; geometry collision mesh filename=stl/lf_lowleg_1.stl scale=0.001 0.001 0.001; visual mesh filename=stl/lf_lowleg_1.stl scale=0.001 0.001 0.001
- link front_left_leg_link: mass 0.1 -> 1.0; geometry collision mesh filename=stl/lf_leg_1.stl scale=0.001 0.001 0.001; visual mesh filename=stl/lf_leg_1.stl scale=0.001 0.001 0.001
- link front_left_leg_link_cover: mass 0.5 -> 0.13180516321676988; geometry collision mesh filename=stl/p2_1.stl scale=0.001 0.001 0.001; visual mesh filename=stl/p2_1.stl scale=0.001 0.001 0.001
- link front_left_shoulder_link: mass 0.10 -> 2.0; geometry collision mesh filename=stl/lf_hip_1.stl scale=0.001 0.001 0.001; visual mesh filename=stl/lf_hip_1.stl scale=0.001 0.001 0.001
- link front_left_toe_link: mass 0.005 -> 0.15329743789754363; geometry collision mesh filename=stl/lf_foot_1.stl scale=0.001 0.001 0.001; visual mesh filename=stl/lf_foot_1.stl scale=0.001 0.001 0.001
- link front_right_foot_link: mass 0.1 -> 0.11741117146712181; geometry collision mesh filename=stl/rf_lowleg_1.stl scale=0.001 0.001 0.001; visual mesh filename=stl/rf_lowleg_1.stl scale=0.001 0.001 0.001
- link front_right_leg_link: mass 0.1 -> 4.39979249324605; geometry collision mesh filename=stl/rf_leg_1.stl scale=0.001 0.001 0.001; visual mesh filename=stl/rf_leg_1.stl scale=0.001 0.001 0.001
- link front_right_leg_link_cover: mass 0.5 -> 0.13180516321676988; geometry collision mesh filename=stl/P4_1.stl scale=0.001 0.001 0.001; visual mesh filename=stl/P4_1.stl scale=0.001 0.001 0.001
- link front_right_shoulder_link: mass 0.10 -> 3.1117770789829353; geometry collision mesh filename=stl/rf_hip_1.stl scale=0.001 0.001 0.001; visual mesh filename=stl/rf_hip_1.stl scale=0.001 0.001 0.001
- link front_right_toe_link: mass 0.005 -> 0.15329743789754363; geometry collision mesh filename=stl/rf_foot_1.stl scale=0.001 0.001 0.001; visual mesh filename=stl/rf_foot_1.stl scale=0.001 0.001 0.001
- link rear_left_foot_link: mass 0.1 -> 0.11741117146712189; geometry collision mesh filename=stl/lh_lowleg_1.stl scale=0.001 0.001 0.001; visual mesh filename=stl/lh_lowleg_1.stl scale=0.001 0.001 0.001
- link rear_left_leg_link: mass 0.10 -> 4.3997924932192625; geometry collision mesh filename=stl/lh_leg_1.stl scale=0.001 0.001 0.001; visual mesh filename=stl/lh_leg_1.stl scale=0.001 0.001 0.001
- link rear_left_leg_link_cover: mass 0.5 -> 0.13180516321676988; geometry collision mesh filename=stl/p1_1.stl scale=0.001 0.001 0.001; visual mesh filename=stl/p1_1.stl scale=0.001 0.001 0.001
- link rear_left_shoulder_link: mass 0.10 -> 3.111777078982937; geometry collision mesh filename=stl/lh_hip_1.stl scale=0.001 0.001 0.001; visual mesh filename=stl/lh_hip_1.stl scale=0.001 0.001 0.001
- link rear_left_toe_link: mass 0.005 -> 0.15329743789754363; geometry collision mesh filename=stl/lh_foot_1.stl scale=0.001 0.001 0.001; visual mesh filename=stl/lh_foot_1.stl scale=0.001 0.001 0.001
- link rear_right_foot_link: mass 0.1 -> 0.11741117146712181; geometry collision mesh filename=stl/rh_lowleg_1.stl scale=0.001 0.001 0.001; visual mesh filename=stl/rh_lowleg_1.stl scale=0.001 0.001 0.001
- link rear_right_leg_link: mass 0.10 -> 4.39979249324605; geometry collision mesh filename=stl/rh_leg_1.stl scale=0.001 0.001 0.001; visual mesh filename=stl/rh_leg_1.stl scale=0.001 0.001 0.001
- link rear_right_leg_link_cover: mass 0.5 -> 0.13180516321676988; geometry collision mesh filename=stl/p3_1.stl scale=0.001 0.001 0.001; visual mesh filename=stl/p3_1.stl scale=0.001 0.001 0.001
- link rear_right_shoulder_link: mass 0.10 -> 3.111777078982936; geometry collision mesh filename=stl/rh_hip_1.stl scale=0.001 0.001 0.001; visual mesh filename=stl/rh_hip_1.stl scale=0.001 0.001 0.001
- link rear_right_toe_link: mass 0.005 -> 0.15329743789754363; geometry collision mesh filename=stl/rh_foot_1.stl scale=0.001 0.001 0.001; visual mesh filename=stl/rh_foot_1.stl scale=0.001 0.001 0.001
Joints:
- removed joint chassis_base_front
- removed joint chassis_base_rear
- joint foot_motor_front_left: axis 0 1 0 -> -0.0 1.0 0.0; limit lower=-0.1 upper=2.59 effort=100.0 velocity=0.5 -> lower=-2.67 upper=2.67 effort=100.0 velocity=0.5; origin xyz=-0.01 0 -0.12 rpy=0 0 0 -> xyz=1.1e-05 0.101005 -0.279173 rpy=0 0 0
- joint foot_motor_front_right: axis 0 1 0 -> -0.0 1.0 -0.0; limit lower=-0.1 upper=2.59 effort=100.0 velocity=0.5 -> lower=-2.67 upper=2.67 effort=100.0 velocity=0.5; origin xyz=-0.01 0 -0.12 rpy=0 0 0 -> xyz=-1.1e-05 -0.101005 -0.279173 rpy=0 0 0
- joint foot_motor_rear_left: axis 0 1 0 -> -0.0 1.0 0.0; limit lower=-0.1 upper=2.59 effort=100.0 velocity=0.5 -> lower=-2.67 upper=2.67 effort=100.0 velocity=0.5; origin xyz=-0.01 0 -0.12 rpy=0 0 0 -> xyz=1.1e-05 0.101005 -0.279173 rpy=0 0 0
- joint foot_motor_rear_right: axis 0 1 0 -> -0.0 1.0 -0.0; limit lower=-0.1 upper=2.59 effort=100.0 velocity=0.5 -> lower=-2.67 upper=2.67 effort=100.0 velocity=0.5; origin xyz=-0.01 0 -0.12 rpy=0 0 0 -> xyz=-1.1e-05 -0.101005 -0.279173 rpy=0 0 0
- joint front_left_leg_cover_joint: origin xyz=0 0 0 -> xyz=0.0 0.105805 0.0 rpy=0 0 0
- joint front_left_toe: origin xyz=0 0 -0.115 -> xyz=0.035728 -0.0042 -0.283561 rpy=0 0 0
- joint front_right_leg_cover_joint: origin xyz=0 0 0 -> xyz=0.0 -0.105805 0.0 rpy=0 0 0
- joint front_right_toe: origin xyz=0 0 -0.115 -> xyz=0.035728 0.0182 -0.283561 rpy=0 0 0
- joint motor_front_left_leg: axis 0 1 0 -> 0.0 1.0 -0.0; limit lower=-2.17 upper=0.97 effort=100.0 velocity=0.5 -> lower=-2.44 upper=2.44 effort=100.0 velocity=0.5; origin xyz=0 -0.052 0 rpy=0 0 0 -> xyz=0.05792 0.03115 0.0 rpy=0 0 0
- joint motor_front_left_shoulder: axis 1 0 0 -> 1.0 0.0 -0.0; limit lower=-1.0 upper=1.0 effort=100.0 velocity=0.7 -> lower=-0.78 upper=0.78 effort=100.0 velocity=0.7; origin xyz=-0.093 -0.036 0 rpy=0 0 0 -> xyz=0.194567 0.048706 0.003592 rpy=0 0 0
- joint motor_front_right_leg: axis 0 1 0 -> -0.0 1.0 -0.0; limit lower=-2.17 upper=0.97 effort=100.0 velocity=0.5 -> lower=-2.44 upper=2.44 effort=100.0 velocity=0.5; origin xyz=0 0.052 0 rpy=0 0 0 -> xyz=0.05792 -0.03115 0.0 rpy=0 0 0
- joint motor_front_right_shoulder: axis 1 0 0 -> 1.0 0.0 -0.0; limit lower=-1.0 upper=1.0 effort=100.0 velocity=0.7 -> lower=-0.78 upper=0.78 effort=100.0 velocity=0.7; origin xyz=-0.093 0.036 0 rpy=0 0 0 -> xyz=0.194567 -0.061294 0.003592 rpy=0 0 0
- joint motor_rear_left_leg: axis 0 1 0 -> 0.0 1.0 0.0; limit lower=-2.17 upper=0.97 effort=100.0 velocity=0.5 -> lower=-2.44 upper=2.44 effort=100.0 velocity=0.5; origin xyz=0 -0.052 0 rpy=0 0 0 -> xyz=-0.05792 0.03115 0.0 rpy=0 0 0
- joint motor_rear_left_shoulder: axis 1 0 0 -> 1.0 -0.0 0.0; limit lower=-1.0 upper=1.0 effort=100.0 velocity=0.7 -> lower=-0.78 upper=0.78 effort=100.0 velocity=0.7; origin xyz=0.093 -0.036 0 rpy=0 0 0 -> xyz=-0.180033 0.048706 0.003592 rpy=0 0 0
- joint motor_rear_right_leg: axis 0 1 0 -> -0.0 1.0 0.0; limit lower=-2.17 upper=0.97 effort=100.0 velocity=0.5 -> lower=-2.44 upper=2.44 effort=100.0 velocity=0.5; origin xyz=0 0.052 0 rpy=0 0 0 -> xyz=-0.05792 -0.03115 0.0 rpy=0 0 0
- joint motor_rear_right_shoulder: axis 1 0 0 -> 1.0 -0.0 0.0; limit lower=-1.0 upper=1.0 effort=100.0 velocity=0.7 -> lower=-0.78 upper=0.78 effort=100.0 velocity=0.7; origin xyz=0.093 0.036 0 rpy=0 0 0 -> xyz=-0.180033 -0.061294 0.003592 rpy=0 0 0
- joint rear_left_leg_cover_joint: origin xyz=0 0 0 -> xyz=0.0 0.105805 0.0 rpy=0 0 0
- joint rear_left_toe: origin xyz=0 0 -0.115 -> xyz=0.035728 -0.0042 -0.283561 rpy=0 0 0
- joint rear_right_leg_cover_joint: origin xyz=0 0 0 -> xyz=0.0 -0.105805 0.0 rpy=0 0 0
- joint rear_right_toe: origin xyz=0 0 -0.115 -> xyz=0.035729 0.0182 -0.283561 rpy=0 0 0

Commit message: Fixing some inertial masses
corrected mass for diffrent parts. Not 100% correct still but close to

File: rex_gym/util/pybullet_data/assets/urdf/rex.urdf (robot description, URDF)
Before this commit: robot rex, 21 links, 20 joints
Links:
- link base_link: mass 10.0 -> 5.0
- link front_right_leg_link: mass 4.39979249324605 -> 1.0
- link front_right_shoulder_link: mass 3.1117770789829353 -> 2.0
- link rear_left_leg_link: mass 4.3997924932192625 -> 1.0
- link rear_left_shoulder_link: mass 3.111777078982937 -> 2.0
- link rear_right_leg_link: mass 4.39979249324605 -> 1.0
- link rear_right_shoulder_link: mass 3.111777078982936 -> 2.0
