Commit message: git checkout rex-gym to mark-ll
works better

File: rex_gym/util/pybullet_data/assets/urdf/backup/rex.urdf (robot description, URDF)
Before this commit: robot rex, 23 links, 22 joints
Links:
- removed link front_left_leg_link_cover
- removed link front_right_leg_link_cover
- removed link rear_left_leg_link_cover
- removed link rear_right_leg_link_cover
- link base_link: mass 1.20 -> 12; geometry collision mesh filename=stl/mainbody.stl scale=0.001 0.001 0.001; visual mesh filename=stl/mainbody.stl scale=0.001 0.001 0.001
- link chassis_front_link: mass 0.05 -> 0.5; geometry collision mesh filename=stl/frontpart.stl scale=0.001 0.001 0.001; visual mesh filename=stl/frontpart.stl scale=0.001 0.001 0.001
- link chassis_rear_link: mass 0.05 -> 0.5; geometry collision mesh filename=stl/backpart.stl scale=0.001 0.001 0.001; visual mesh filename=stl/backpart.stl scale=0.001 0.001 0.001
- link front_left_foot_link: mass 0.1 -> 0.25; geometry collision mesh filename=stl/lower_leg_solid.stl scale=0.001 0.001 0.001; visual mesh filename=stl/lower_leg_solid.stl scale=0.001 0.001 0.001
- link front_left_leg_link: mass 0.1 -> 1.5; geometry collision mesh filename=stl/upper_leg.stl scale=0.001 0.001 0.001; visual mesh filename=stl/upper_leg.stl scale=0.001 0.001 0.001
- link front_left_shoulder_link: mass 0.10 -> 1; geometry collision mesh filename=stl/shoulder.stl scale=0.001 0.001 0.001; visual mesh filename=stl/shoulder.stl scale=0.001 0.001 0.001
- link front_left_toe_link: mass 0.005 -> 0.01
- link front_right_foot_link: mass 0.1 -> 0.25; geometry collision mesh filename=stl/lower_leg_solid.stl scale=0.001 0.001 0.001; visual mesh filename=stl/lower_leg_solid.stl scale=0.001 0.001 0.001
- link front_right_leg_link: mass 0.1 -> 1.5; geometry collision mesh filename=stl/upper_leg.stl scale=0.001 0.001 0.001; visual mesh filename=stl/upper_leg.stl scale=0.001 0.001 0.001
- link front_right_shoulder_link: mass 0.10 -> 1; geometry collision mesh filename=stl/shoulder.stl scale=0.001 0.001 0.001; visual mesh filename=stl/shoulder.stl scale=0.001 0.001 0.001
- link front_right_toe_link: mass 0.005 -> 0.01
- link rear_left_foot_link: mass 0.1 -> 0.25; geometry collision mesh filename=stl/lower_leg_solid.stl scale=0.001 0.001 0.001; visual mesh filename=stl/lower_leg_solid.stl scale=0.001 0.001 0.001
- link rear_left_leg_link: mass 0.10 -> 1.5; geometry collision mesh filename=stl/upper_leg.stl scale=0.001 0.001 0.001; visual mesh filename=stl/upper_leg.stl scale=0.001 0.001 0.001
- link rear_left_shoulder_link: mass 0.10 -> 1; geometry collision mesh filename=stl/shoulder.stl scale=0.001 0.001 0.001; visual mesh filename=stl/shoulder.stl scale=0.001 0.001 0.001
- link rear_left_toe_link: mass 0.005 -> 0.01
- link rear_right_foot_link: mass 0.1 -> 0.25; geometry collision mesh filename=stl/lower_leg_solid.stl scale=0.001 0.001 0.001; visual mesh filename=stl/lower_leg_solid.stl scale=0.001 0.001 0.001
- link rear_right_leg_link: mass 0.10 -> 1.5; geometry collision mesh filename=stl/upper_leg.stl scale=0.001 0.001 0.001; visual mesh filename=stl/upper_leg.stl scale=0.001 0.001 0.001
- link rear_right_shoulder_link: mass 0.10 -> 1; geometry collision mesh filename=stl/shoulder.stl scale=0.001 0.001 0.001; visual mesh filename=stl/shoulder.stl scale=0.001 0.001 0.001
- link rear_right_toe_link: mass 0.005 -> 0.01
Joints:
- removed joint front_left_leg_cover_joint
- removed joint front_left_toe
- removed joint front_right_leg_cover_joint
- removed joint front_right_toe
- removed joint rear_left_leg_cover_joint
- removed joint rear_left_toe
- removed joint rear_right_leg_cover_joint
- removed joint rear_right_toe
- added joint toe_joint_front_left: type fixed, parent front_left_foot_link, child front_left_toe_link, origin xyz=0 -0.0098 -0.16
- added joint toe_joint_front_right: type fixed, parent front_right_foot_link, child front_right_toe_link, origin xyz=0 -0.0098 -0.16
- added joint toe_joint_rear_left: type fixed, parent rear_left_foot_link, child rear_left_toe_link, origin xyz=0 -0.0098 -0.16
- added joint toe_joint_rear_right: type fixed, parent rear_right_foot_link, child rear_right_toe_link, origin xyz=0 -0.0098 -0.16
- joint chassis_base_front: origin (none) -> xyz=-0.042 -0.055 -0.01 rpy=0 0 0
- joint chassis_base_rear: origin (none) -> xyz=0.05 0 -0.038 rpy=0 0 0
- joint foot_motor_front_left: limit lower=-0.1 upper=2.59 effort=100.0 velocity=0.5 -> lower=-3.14 upper=3.14 effort=100.0 velocity=100; origin xyz=-0.01 0 -0.12 rpy=0 0 0 -> xyz=0 -0.047 -0.16 rpy=0 0 0
- joint foot_motor_front_right: limit lower=-0.1 upper=2.59 effort=100.0 velocity=0.5 -> lower=-3.14 upper=3.14 effort=100.0 velocity=100; origin xyz=-0.01 0 -0.12 rpy=0 0 0 -> xyz=0 0.047 -0.16 rpy=0 0 0
- joint foot_motor_rear_left: limit lower=-0.1 upper=2.59 effort=100.0 velocity=0.5 -> lower=-3.14 upper=3.14 effort=100.0 velocity=100; origin xyz=-0.01 0 -0.12 rpy=0 0 0 -> xyz=0 -0.047 -0.16 rpy=0 0 0
- joint foot_motor_rear_right: limit lower=-0.1 upper=2.59 effort=100.0 velocity=0.5 -> lower=-3.14 upper=3.14 effort=100.0 velocity=100; origin xyz=-0.01 0 -0.12 rpy=0 0 0 -> xyz=0 0.047 -0.16 rpy=0 0 0
- joint motor_front_left_leg: limit lower=-2.17 upper=0.97 effort=100.0 velocity=0.5 -> lower=-1.57 upper=1.57 effort=100.0 velocity=100; origin xyz=0 -0.052 0 rpy=0 0 0 -> xyz=0 -0.017 0 rpy=0 0 0
- joint motor_front_left_shoulder: limit lower=-1.0 upper=1.0 effort=100.0 velocity=0.7 -> lower=-1.0 upper=1.0 effort=100.0 velocity=100; origin xyz=-0.093 -0.036 0 rpy=0 0 0 -> xyz=-0.095 -0.035 0 rpy=0 0 0
- joint motor_front_right_leg: limit lower=-2.17 upper=0.97 effort=100.0 velocity=0.5 -> lower=-1.57 upper=1.57 effort=100.0 velocity=100; origin xyz=0 0.052 0 rpy=0 0 0 -> xyz=0 0.017 0 rpy=0 0 0
- joint motor_front_right_shoulder: limit lower=-1.0 upper=1.0 effort=100.0 velocity=0.7 -> lower=-1.0 upper=1.0 effort=100.0 velocity=100; origin xyz=-0.093 0.036 0 rpy=0 0 0 -> xyz=-0.095 0.035 0 rpy=0 0 0
- joint motor_rear_left_leg: limit lower=-2.17 upper=0.97 effort=100.0 velocity=0.5 -> lower=-1.57 upper=1.57 effort=100.0 velocity=100; origin xyz=0 -0.052 0 rpy=0 0 0 -> xyz=0 -0.017 0 rpy=0 0 0
- joint motor_rear_left_shoulder: limit lower=-1.0 upper=1.0 effort=100.0 velocity=0.7 -> lower=-1.0 upper=1.0 effort=100.0 velocity=100; origin xyz=0.093 -0.036 0 rpy=0 0 0 -> xyz=0.09 -0.035 0 rpy=0 0 0
- joint motor_rear_right_leg: limit lower=-2.17 upper=0.97 effort=100.0 velocity=0.5 -> lower=-1.57 upper=1.57 effort=100.0 velocity=100; origin xyz=0 0.052 0 rpy=0 0 0 -> xyz=0 0.017 0 rpy=0 0 0
- joint motor_rear_right_shoulder: limit lower=-1.0 upper=1.0 effort=100.0 velocity=0.7 -> lower=-1.0 upper=1.0 effort=100.0 velocity=100; origin xyz=0.093 0.036 0 rpy=0 0 0 -> xyz=0.09 0.035 0 rpy=0 0 0

File: rex_gym/util/pybullet_data/assets/urdf/rex.urdf (robot description, URDF)
Before this commit: robot rex, 21 links, 20 joints
Links:
- link base_link: mass 5.0 -> 6.0

File: rex_gym/util/pybullet_data/assets/urdf/rex_arm.urdf (robot description, URDF)
Before this commit: robot rex_arm, 31 links, 30 joints
Links:
- added link arm_section_1_ext, mass 0; collision cylinder length=0.05 radius=0.02; visual mesh filename=meshes/section_1.obj
- added link arm_section_4_ext, mass 0; collision cylinder length=0.05 radius=0.02; visual mesh filename=meshes/section_4.obj
- link arm_fixed_tip: mass 0.05 -> 0
- link arm_long_U: mass 1. -> 0
- link arm_moving_tip: mass 0.05 -> 0
- link arm_section_1: mass 0.2 -> 0
- link arm_section_2: mass 0.2 -> 0
- link arm_section_3: mass 0.2 -> 0
- link arm_section_4: mass 0.2 -> 0; geometry collision cylinder length=0.05 radius=0.02; visual mesh filename=meshes/section_2.obj
- link arm_section_5: mass 0.2 -> 0
- link front_left_foot_link: geometry collision box size=0.026 0.020 0.115; visual mesh filename=stl/lower_leg_solid.stl scale=0.001 0.001 0.001
- link front_left_leg_link: geometry collision box size=0.028 0.036 0.12; visual mesh filename=stl/upper_leg_shell_base.stl scale=0.001 0.001 0.001
- link front_left_leg_link_cover: geometry visual mesh filename=stl/upper_leg_shell_cover.stl scale=0.001 0.001 0.001
- link front_right_foot_link: geometry collision box size=0.026 0.020 0.115; visual mesh filename=stl/lower_leg_solid.stl scale=0.001 0.001 0.001
- link front_right_leg_link: geometry collision box size=0.028 0.036 0.12; visual mesh filename=stl/upper_leg_shell_base.stl scale=0.001 0.001 0.001
- link front_right_leg_link_cover: geometry visual mesh filename=stl/upper_leg_shell_cover.stl scale=0.001 0.001 0.001
- link rear_left_foot_link: geometry collision box size=0.026 0.020 0.115; visual mesh filename=stl/lower_leg_solid.stl scale=0.001 0.001 0.001
- link rear_left_leg_link: geometry collision box size=0.028 0.036 0.12; visual mesh filename=stl/upper_leg_shell_base.stl scale=0.001 0.001 0.001
- link rear_left_leg_link_cover: geometry visual mesh filename=stl/upper_leg_shell_cover.stl scale=0.001 0.001 0.001
- link rear_right_foot_link: geometry collision box size=0.026 0.020 0.115; visual mesh filename=stl/lower_leg_solid.stl scale=0.001 0.001 0.001
- link rear_right_leg_link: geometry collision box size=0.028 0.036 0.12; visual mesh filename=stl/upper_leg_shell_base.stl scale=0.001 0.001 0.001
- link rear_right_leg_link_cover: geometry visual mesh filename=stl/upper_leg_shell_cover.stl scale=0.001 0.001 0.001
Joints:
- removed joint front_left_toe
- removed joint front_right_toe
- removed joint rear_left_toe
- removed joint rear_right_toe
- added joint arm_1_ext: type fixed, parent arm_section_1, child arm_section_1_ext, origin xyz=0.048 0 0 rpy=0 1.5707963267949 0, axis 0 0 1
- added joint motor_arm_m7: type revolute, parent arm_section_4_ext, child arm_section_5, origin xyz=0 0 0 rpy=0 0 0, axis 0 0 -1, limit lower=-0.436 upper=1.5 effort=100.0 velocity=0.7
- added joint toe_joint_front_left: type fixed, parent front_left_foot_link, child front_left_toe_link, origin xyz=0 0 -0.115
- added joint toe_joint_front_right: type fixed, parent front_right_foot_link, child front_right_toe_link, origin xyz=0 0 -0.115
- added joint toe_joint_rear_left: type fixed, parent rear_left_foot_link, child rear_left_toe_link, origin xyz=0 0 -0.115
- added joint toe_joint_rear_right: type fixed, parent rear_right_foot_link, child rear_right_toe_link, origin xyz=0 0 -0.115
- joint arm_t7f: origin xyz=0 -0.11 0 rpy=-1.5707963267949 0 0 -> xyz=0 0 0 rpy=0 0 0; parent arm_section_4 -> arm_section_4_ext
- joint foot_motor_front_left: limit lower=-0.1 upper=2.59 effort=100.0 velocity=0.5 -> lower=-3.14 upper=3.14 effort=100.0 velocity=0.5; origin xyz=-0.01 0 -0.12 rpy=0 0 0 -> xyz=0.002 -0.02 -0.16 rpy=0 0 0
- joint foot_motor_front_right: limit lower=-0.1 upper=2.59 effort=100.0 velocity=0.5 -> lower=-3.14 upper=3.14 effort=100.0 velocity=0.5; origin xyz=-0.01 0 -0.12 rpy=0 0 0 -> xyz=0.002 0.02 -0.16 rpy=0 0 0
- joint foot_motor_rear_left: limit lower=-0.1 upper=2.59 effort=100.0 velocity=0.5 -> lower=-3.14 upper=3.14 effort=100.0 velocity=0.5; origin xyz=-0.01 0 -0.12 rpy=0 0 0 -> xyz=0.002 -0.02 -0.16 rpy=0 0 0
- joint foot_motor_rear_right: limit lower=-0.1 upper=2.59 effort=100.0 velocity=0.5 -> lower=-3.14 upper=3.14 effort=100.0 velocity=0.5; origin xyz=-0.01 0 -0.12 rpy=0 0 0 -> xyz=0.002 0.02 -0.16 rpy=0 0 0
- joint motor_arm_m1: limit lower=-1.5 upper=1.5 effort=100.0 velocity=0.7 -> lower=-4.71 upper=1.57 effort=100.0 velocity=0.5; origin xyz=-0.03 0 0.0327993216120967 rpy=0 0 0 -> xyz=-0.05 -0.005 0.0327993216120967 rpy=0 0 0
- joint motor_arm_m2: limit lower=-1.5 upper=1.5 effort=100.0 velocity=0.7 -> lower=-1.57 upper=1.57 effort=100.0 velocity=0.5
- joint motor_arm_m3: limit lower=-1.5 upper=1.5 effort=100.0 velocity=0.7 -> lower=-1.57 upper=1.57 effort=100.0 velocity=0.5; origin xyz=0.054 0 0 rpy=0 0 0 -> xyz=0.1 0 0 rpy=0 0 0
- joint motor_arm_m4: limit lower=-1.5 upper=1.5 effort=100.0 velocity=0.7 -> lower=-3.14 upper=3.14 effort=100.0 velocity=0.5
- joint motor_arm_m5: axis 0 0 1 -> 1 0 0; limit lower=-1.5 upper=1.5 effort=100.0 velocity=0.7 -> lower=-1.57 upper=1.57 effort=100.0 velocity=0.5; origin xyz=0 -0.048 0 rpy=0 -1.5707963267949 0 -> xyz=0 -0.048 0 rpy=-1.57 0 3.14
- joint motor_arm_m6: axis 0 0 -1 -> 0 1 0; child arm_section_5 -> arm_section_4_ext; limit lower=-1.3 upper=.2 effort=100.0 velocity=0.7 -> lower=-1.57 upper=1.57 effort=100.0 velocity=0.5; origin xyz=0 -0.058 0 rpy=0 -1.5707963267949 0 -> xyz=0 0 0.097 rpy=-1.57 0 0
- joint motor_front_left_leg: limit lower=-2.17 upper=0.97 effort=100.0 velocity=0.5 -> lower=-1.57 upper=1.57 effort=100.0 velocity=0.5
- joint motor_front_right_leg: limit lower=-2.17 upper=0.97 effort=100.0 velocity=0.5 -> lower=-1.57 upper=1.57 effort=100.0 velocity=0.5; origin xyz=0 0.052 0 rpy=0 0 0 -> xyz=0 0.042 0 rpy=0 0 0
- joint motor_rear_left_leg: limit lower=-2.17 upper=0.97 effort=100.0 velocity=0.5 -> lower=-1.57 upper=1.57 effort=100.0 velocity=0.5
- joint motor_rear_right_leg: limit lower=-2.17 upper=0.97 effort=100.0 velocity=0.5 -> lower=-1.57 upper=1.57 effort=100.0 velocity=0.5; origin xyz=0 0.052 0 rpy=0 0 0 -> xyz=0 0.042 0 rpy=0 0 0
